Commit message: navigation nodes (ex-move_base) use ground truth odom and scan

File: airlab/gazebo/robot_realistic.urdf (robot description, URDF)
Before this commit: robot turtlebot3_waffle, 13 links, 12 joints
Links:
- removed link base_footprint
- removed link base_link
- removed link base_scan
- removed link camera_depth_frame
- removed link camera_depth_optical_frame
- removed link camera_link
- removed link camera_rgb_frame
- removed link camera_rgb_optical_frame
- removed link caster_back_left_link
- removed link caster_back_right_link
- removed link imu_link
- removed link wheel_left_link
- removed link wheel_right_link
- added link base_footprint_realistic
- added link base_link_realistic, mass 1.3729096e+00; collision box size=0.266 0.266 0.094; visual mesh filename=package://turtlebot3_description/meshes/bases/waffle_base.s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 scale=0.001 0.001 0.001
- added link base_scan_realistic, mass 0.114; collision cylinder length=0.0315 radius=0.055; visual mesh filename=package://turtlebot3_description/meshes/sensors/lds.stl scale=0.001 0.001 0.001
- added link camera_depth_frame_realistic
- added link camera_depth_optical_frame_realistic
- added link camera_link_realistic; collision box size=0.012 0.132 0.020; visual mesh filename=package://turtlebot3_description/meshes/sensors/r200.dae
- added link camera_rgb_frame_realistic
- added link camera_rgb_optical_frame_realistic
- added link caster_back_left_link_realistic, mass 0.005; collision box size=0.030 0.009 0.020
- added link caster_back_right_link_realistic, mass 0.005; collision box size=0.030 0.009 0.020
- added link imu_link_realistic
- added link wheel_left_link_realistic, mass 2.8498940e-02; collision cylinder length=0.018 radius=0.033; visual mesh filename=package://turtlebot3_description/meshes/wheels/left_tire.stl scale=0.001 0.001 0.001
- added link wheel_right_link_realistic, mass 2.8498940e-02; collision cylinder length=0.018 radius=0.033; visual mesh filename=package://turtlebot3_description/meshes/wheels/right_tire.s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 scale=0.001 0.001 0.001
Joints:
- joint base_joint: child base_link -> base_link_realistic; parent base_footprint -> base_footprint_realistic
- joint camera_depth_joint: child camera_depth_frame -> camera_depth_frame_realistic; parent camera_link -> camera_link_realistic
- joint camera_depth_optical_joint: child camera_depth_optical_frame -> camera_depth_optical_frame_realistic; parent camera_depth_frame -> camera_depth_frame_realistic
- joint camera_joint: child camera_link -> camera_link_realistic; parent base_link -> base_link_realistic
- joint camera_rgb_joint: child camera_rgb_frame -> camera_rgb_frame_realistic; parent camera_link -> camera_link_realistic
- joint camera_rgb_optical_joint: child camera_rgb_optical_frame -> camera_rgb_optical_frame_realistic; parent camera_rgb_frame -> camera_rgb_frame_realistic
- joint caster_back_left_joint: child caster_back_left_link -> caster_back_left_link_realistic; parent base_link -> base_link_realistic
- joint caster_back_right_joint: child caster_back_right_link -> caster_back_right_link_realistic; parent base_link -> base_link_realistic
- joint imu_joint: child imu_link -> imu_link_realistic; parent base_link -> base_link_realistic
- joint scan_joint: child base_scan -> base_scan_realistic; parent base_link -> base_link_realistic
- joint wheel_left_joint: child wheel_left_link -> wheel_left_link_realistic; parent base_link -> base_link_realistic
- joint wheel_right_joint: child wheel_right_link -> wheel_right_link_realistic; parent base_link -> base_link_realistic
