Commit message: updated to dataset v4

File: airlab/gazebo/robot.urdf (robot description, URDF)
Before this commit: robot turtlebot3_waffle, 13 links, 12 joints
Links:
- removed link base_footprint_realistic
- removed link base_link_realistic
- removed link base_scan_realistic
- removed link camera_depth_frame_realistic
- removed link camera_depth_optical_frame_realistic
- removed link camera_link_realistic
- removed link camera_rgb_frame_realistic
- removed link camera_rgb_optical_frame_realistic
- removed link caster_back_left_link_realistic
- removed link caster_back_right_link_realistic
- removed link imu_link_realistic
- removed link wheel_left_link_realistic
- removed link wheel_right_link_realistic
- added link base_footprint
- added link base_link, mass 1.3729096e+00; collision box size=0.266 0.266 0.094; visual mesh filename=package://turtlebot3_description/meshes/bases/waffle_base.s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 scale=0.001 0.001 0.001
- added link base_scan, mass 0.114; collision cylinder length=0.0315 radius=0.055; visual mesh filename=package://turtlebot3_description/meshes/sensors/lds.stl scale=0.001 0.001 0.001
- added link camera_depth_frame
- added link camera_depth_optical_frame
- added link camera_link; collision box size=0.012 0.132 0.020; visual mesh filename=package://turtlebot3_description/meshes/sensors/r200.dae
- added link camera_rgb_frame
- added link camera_rgb_optical_frame
- added link caster_back_left_link, mass 0.005; collision box size=0.030 0.009 0.020
- added link caster_back_right_link, mass 0.005; collision box size=0.030 0.009 0.020
- added link imu_link
- added link wheel_left_link, mass 2.8498940e-02; collision cylinder length=0.018 radius=0.033; visual mesh filename=package://turtlebot3_description/meshes/wheels/left_tire.stl scale=0.001 0.001 0.001
- added link wheel_right_link, mass 2.8498940e-02; collision cylinder length=0.018 radius=0.033; visual mesh filename=package://turtlebot3_description/meshes/wheels/right_tire.s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 scale=0.001 0.001 0.001
Joints:
- joint base_joint: child base_link_realistic -> base_link; parent base_footprint_realistic -> base_footprint
- joint camera_depth_joint: child camera_depth_frame_realistic -> camera_depth_frame; parent camera_link_realistic -> camera_link
- joint camera_depth_optical_joint: child camera_depth_optical_frame_realistic -> camera_depth_optical_frame; parent camera_depth_frame_realistic -> camera_depth_frame
- joint camera_joint: child camera_link_realistic -> camera_link; parent base_link_realistic -> base_link
- joint camera_rgb_joint: child camera_rgb_frame_realistic -> camera_rgb_frame; parent camera_link_realistic -> camera_link
- joint camera_rgb_optical_joint: child camera_rgb_optical_frame_realistic -> camera_rgb_optical_frame; parent camera_rgb_frame_realistic -> camera_rgb_frame
- joint caster_back_left_joint: child caster_back_left_link_realistic -> caster_back_left_link; parent base_link_realistic -> base_link
- joint caster_back_right_joint: child caster_back_right_link_realistic -> caster_back_right_link; parent base_link_realistic -> base_link
- joint imu_joint: child imu_link_realistic -> imu_link; parent base_link_realistic -> base_link
- joint scan_joint: child base_scan_realistic -> base_scan; parent base_link_realistic -> base_link
- joint wheel_left_joint: child wheel_left_link_realistic -> wheel_left_link; parent base_link_realistic -> base_link
- joint wheel_right_joint: child wheel_right_link_realistic -> wheel_right_link; parent base_link_realistic -> base_link
