Commit message: robot models and dataset

File: robots/hunter2/robot.urdf (robot description, URDF)
Before this commit: robot turtlebot3_waffle, 3 links, 1 joints
Links:
- removed link chassis
- removed link odom_demo
- added link base_footprint
- added link base_scan, mass 0.125; collision cylinder length=0.055 radius=0.0508; visual mesh filename=package://turtlebot3_description/meshes/sensors/lds.stl scale=0.001 0.001 0.001
- link base_link: mass 1.3729096e+00 -> None; geometry 
Joints:
- removed joint base_joint
- added joint joint_footprint: type fixed, parent base_link, child base_footprint, origin xyz=0 0 0 rpy=0 0 0
- added joint scan_joint: type fixed, parent base_link, child base_scan, origin xyz=0.325 0.115 0.35 rpy=0 0 0

Commit message: fixed everything

File: robots/hunter2/robot.urdf (robot description, URDF)
Before this commit: robot hunter_v2, 3 links, 2 joints
Links:
- link base_scan: mass 0.125 -> None; geometry 
Joints:
- joint joint_footprint: origin xyz=0 0 0 rpy=0 0 0 -> xyz=0 0 -0.166 rpy=0 0 0
- joint scan_joint: origin xyz=0.325 0.115 0.35 rpy=0 0 0 -> xyz=0.325 0.115 0.29 rpy=0 0 0
